File: Amstrad-PCW8xxx.kicad_pcb (KiCad board)
At the start: 2 copper layers, 265.1 x 155.1 mm, 110 parts, among them IC101 GateArray, IC102 Z80A, IC103 74HCU04, IC104 TMM41256AP, IC105 TMM41256AP, IC106 TMM41256AP, IC107 TMM41256AP, IC108 TMM41256AP, IC109 TMM41256AP, IC110 TMM41256AP, IC111 TMM41256AP, IC112 TMM41256AP, IC113 TMM41256AP, IC114 TMM41256AP, IC115 TMM41256AP, IC116 TMM41256AP, IC117 TMM41256AP, IC118 TMM41256AP, IC119 TMM41256AP, IC120 TC74HC14, IC201 SED9420AC, IC202 74HC00, IC203 D765AC-2, IC204 74HC04, IC205 74HC04, IC701 40026, X101 32MHz, X201 18MHz, X701 11MHz

Commit message: progress PCB layout
Parts:
- C101, C102, C103, C104, C105, C106, C107, C108, C109, C110, C111, C112, C113, C114, C115, C116, C117, C118, C119, C120, C126, C127, C128, C201, C202, C203, C204, C205, C206, C207, C208, C209, C210, C701, C702, C703: footprint Capacitor_THT:C_Disc_D10.0mm_W2.5mm_P5.00mm -> Library:C_Disc_D9.0mm_W2.5mm_P5.00mm
- moved C111 113.9 mm to (136.3, 142.2), turned to -90 degrees
- moved C110 112.2 mm to (136.3, 132.0), turned to -90 degrees
- moved C109 110.8 mm to (136.3, 121.8), turned to -90 degrees
- moved C108 109.8 mm to (136.3, 111.7), turned to -90 degrees
- moved C107 109.1 mm to (136.3, 101.5), turned to -90 degrees
- moved C104 109.0 mm to (136.3, 71.0), turned to -90 degrees
- moved C106 108.7 mm to (136.3, 91.3), turned to -90 degrees
- moved C105 108.7 mm to (136.3, 81.2), turned to -90 degrees
- moved C112 93.2 mm to (111.1, 71.0), turned to -90 degrees
- moved C119 87.8 mm to (111.1, 142.2), turned to -90 degrees
- moved C118 84.4 mm to (111.1, 132.0), turned to -90 degrees
- moved C117 81.4 mm to (111.1, 121.8), turned to -90 degrees
- moved C116 78.7 mm to (111.1, 111.7), turned to -90 degrees
- moved C115 76.4 mm to (111.1, 101.5), turned to -90 degrees
- moved C114 74.6 mm to (111.1, 91.3), turned to -90 degrees
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Other:
- outline, holes or cut-outs redrawn

Commit message: layout pcb components
Parts:
- added C121: 10V47uF, Capacitor_THT:CP_Radial_D10.0mm_P5.00mm, F.Cu at (98.0, 91.7)
- added D101: 1S2472, Library:D_DO-35_SOD27_P10.16mm_Horizontal, F.Cu at (165.9, 133.3)
- added D102: ~, Diode_THT:D_DO-35_SOD27_P10.16mm_Horizontal, F.Cu at (321.8, 83.5)
- added D103: ~, Diode_THT:D_DO-35_SOD27_P10.16mm_Horizontal, F.Cu at (314.2, 87.3)
- added R121: 2K2, Library:R_Axial_DIN0207_L6.3mm_D2.5mm_P10.16mm_Horizontal, F.Cu at (290.8, 74.9)
- C123: footprint Capacitor_THT:CP_Radial_D10.0mm_P5.00mm -> Library:C_Disc_D9.0mm_W2.5mm_P5.00mm
- R101, R102, R103, R104, R105, R106, R107, R108, R109, R110, R111, R112, R113, R114, R115, R116, R117, R118, R119, R120, R122, R123, R124, R201, R202, R203, R204, R206, R701, R725: footprint Resistor_THT:R_Axial_DIN0207_L6.3mm_D2.5mm_P10.16mm_Horizontal -> Library:R_Axial_DIN0207_L6.3mm_D2.5mm_P10.16mm_Horizontal
- moved C102 268.1 mm to (295.0, 89.8), turned to 180 degrees
- moved C122 266.1 mm to (97.9, 84.3)
- moved C123 266.1 mm to (98.1, 73.9)
- moved CP103 258.4 mm to (328.1, 80.9), turned to 90 degrees
- moved C128 258.3 mm to (306.5, 93.6), turned to 180 degrees
- moved CP706 255.8 mm to (112.5, 56.4), turned to 90 degrees
- moved CP101 243.2 mm to (328.1, 106.3), turned to 90 degrees
- moved IC112 237.4 mm to (310.4, 192.7), turned to 90 degrees
- moved C103 233.3 mm to (258.3, 110.0), turned to -90 degrees
- moved C112 229.6 mm to (306.6, 191.4), turned to 90 degrees
- moved IC113 227.6 mm to (310.4, 182.6), turned to 90 degrees
- moved C126 226.7 mm to (265.6, 121.9), turned to 180 degrees
- moved R101 225.9 mm to (100.1, 152.4), turned to -90 degrees
- moved C127 224.3 mm to (265.6, 117.9), turned to 180 degrees
- moved IC120 220.3 mm to (301.5, 74.3), turned to 0 degrees
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Other:
- outline, holes or cut-outs redrawn

Commit message: finish up PCB layout
Parts:
- removed NR107: 10K, Resistor_THT:R_Array_SIP5
- added CP100: Power Supply Connection, Library:Power Connection, F.Cu at (99.8, 126.5)
- added J101: Printer Power, Connector_BarrelJack:BarrelJack_Horizontal, F.Cu at (85.9, 56.6)
- added L101: 2.2uH, Inductor_THT:L_Axial_L6.6mm_D2.7mm_P10.16mm_Horizontal_Vishay_IM-2, F.Cu at (258.3, 127.1)
- added LK1: ~, Library:Link_2, F.Cu at (182.1, 117.5)
- added LS1: Speaker, Library:Speaker, F.Cu at (100.3, 182.5)
- C121, C122, C124: footprint Capacitor_THT:CP_Radial_D10.0mm_P5.00mm -> Library:CP_Radial_P5.00mm
- CD203: footprint Connector_IDC:IDC-Header_2x13_P2.54mm_Horizontal -> Connector_IDC:IDC-Header_2x13_P2.54mm_Vertical
- IC101: footprint Package_QFP:Hitachi_FP80B_PQFP-80_14x20mm_P0.8mm -> Library:Amstrad_PQFP-80_14x20mm_P0.8mm
- IC201: footprint Package_DIP:DIP-24_18.0mmx34.29mm_W15.24mm -> Package_DIP:DIP-28_W15.24mm
- NR202: footprint Resistor_THT:R_Array_SIP6 -> Resistor_THT:R_Array_SIP8
- moved CP706 7.17 mm to (105.9, 53.6)
- moved IC201 3.57 mm to (115.8, 133.6)
- moved CD203 1.57 mm to (231.9, 192.8)
- moved NR202 0.37 mm to (199.0, 186.1)
- moved IC101 0.11 mm to (211.2, 144.6)
Connections:
- NR102 pad 2: (no net) -> /E40
- NR102 pad 3: (no net) -> /E42
- NR102 pad 4: (no net) -> /E34
- NR102 pad 5: (no net) -> /E41
Other:
- outline, holes or cut-outs redrawn
